File: hardware/v1.6/pc_sensything_v1.6/pc_sensything_v1.6.kicad_pcb (KiCad board)
At the start: 4 copper layers, 47 x 57 mm, 102 parts, among them IC1 ESP32-PICO-D4, J1 Qwiic1, J4 Qwiic2, Q1 MBT3904DW1T1, Q2 2.5A/30V, Q3 2.5A/30V, SW2 KMR2, U1 FTS31XS-U, U3 MCP73831, U8 AP2112K-3.3V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

Commit message: Sketches running on Sensything.
Other:
- copper layers 4 -> 2
